File: Display101Adapter.kicad_pcb (KiCad board)
At the start: 2 copper layers, 30.7 x 57.6 mm, 8 parts, among them J1 FFC3B07-40-T, J2 ER-TFTM101 header, J21 Display, SW1 Display Reset

Commit message: v3.0 added
Parts:
- added REF**: MountingHole_3.2mm_M3, MountingHole:MountingHole_3.2mm_M3, F.Cu at (138.5, 126.6)
- added REF**: MountingHole_3.2mm_M3, MountingHole:MountingHole_3.2mm_M3, F.Cu at (163.2, 68.7)
- added REF**: MountingHole_3.2mm_M3, MountingHole:MountingHole_3.2mm_M3, F.Cu at (163.3, 126.5)
- added REF**: MountingHole_3.2mm_M3, MountingHole:MountingHole_3.2mm_M3, F.Cu at (138.6, 68.6)
- J1: moved to F.Cu
- JP1, JP2, JP3, JP4: moved to B.Cu
- moved JP4 13.4 mm to (149.5, 81.0), turned to 0 degrees
- moved J1 12.3 mm to (162.7, 97.6)
- moved J21 8.42 mm to (150.4, 91.3)
- moved JP1 8.19 mm to (144.8, 93.5)
- moved JP2 4.21 mm to (145.0, 109.3)
- moved JP3 3.16 mm to (149.6, 119.0)
- moved SW1 2.52 mm to (153.3, 125.8)
Routing:
- net +VIN: track 68.5 -> 113.2 mm, vias 0 -> 1
- net T_RST: track 34.7 -> 50.8 mm
- net D_BL: track 20.3 -> 35.9 mm
- net D_SDO/RX: track 42.2 -> 32.1 mm, vias 0 -> 1
- net T_INT: track 21.7 -> 30.4 mm
- net D_RST: track 58.0 -> 66.1 mm, vias 1 -> 0
- net D_CLK: track 39.0 -> 33.5 mm, vias 0 -> 1
- net GP13: track 43.7 -> 39.8 mm, vias 2 -> 1
- net GND: track 33.6 -> 29.7 mm, vias 0 -> 3
- net D_CS: track 33.0 -> 35.5 mm
- net GP12: track 32.9 -> 34.6 mm, vias 2 -> 1
- net GP14: track 10.4 -> 11.8 mm
- net D_SDI/TX: track 38.9 -> 37.5 mm
- net Net-(JP3-C): track 8.39 -> 7.23 mm
- added copper zone on F.Cu, net GND
- removed copper zone on F.Cu, net +VIN
Other:
- board size 30.7 x 57.6 mm -> 32 x 65 mm
- board text added: "SPI Display Adapter V 1.3"
- board text removed: "Display Adapter V 1.1"
- board text removed: "GND Data +5v GND"
