File: LCC-Pico-Node_v3_0C - 0805.kicad_sch (KiCad schematic)
At the start: 85 parts, among them IC1 TPS54228DR, IC2 MCP2518FD, IC3 MCP2562FD, IC5 MB85RCxxxV, IC6 TPS54228DR, J1 RJ45, J12 Power Sel, J15 Analog I/O, J16 NVM Power Sel, J2 RJ45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

Commit message: Production level
0805 boards can be assembled at JLCPCB with these files
1206 boards are for hand assembly
Parts:
- C1, C10, C11, C12, C13, C14, C15, C16, C17, C18, C19, C22, C3, C4, C5, C6, C7, C8, C9: footprint Capacitor_SMD:C_1206_3216Metric -> Capacitor_SMD:C_0805_2012Metric
- D1, D12, D4, D5, D7, D8: footprint LED_SMD:LED_1206_3216Metric -> LED_SMD:LED_0805_2012Metric
- F1, F2: value 0ZCG0035AF2C -> 0ZCG0050AF2C; LCSC C3762402 -> C3762102; Manufacturer_Part_Number 0ZCG0035AF2C -> 0ZCG0050AF2C; Mouser Part Number 530-0ZCG0035AF2C -> 530-0ZCG0050AF2C
- IC5: value MB85RCxxxV -> 256Kb; Description_1 FUJITSU - MB85RC256VPNF-G-JNE1 - FRAM, 256KBIT, I2C, SOP-8 -> EEPROM ICs, Memory, 256KBit, I&sup2;C BUS, High Endurance, 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; LCSC C2062875 -> C90485; Manufacturer_Name Fujitsu Semiconductor -> ROHM Semiconductor; Manufacturer_Part_Number MB85RC256VPNF-G-JNE1 -> BR24G256F-5E2; Mouser Part Number 249-MB85RC256VPNJNE1 -> 755-BR24G256F-5E2; Mouser Price/Stock https://www.mouser.co.uk/ProductDetail/Fujitsu-Semiconducto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 -> https://www.mouser.com/ProductDetail/ROHM-Semiconductor/BR2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
- J20: LCSC (none) -> C431534
- JP2, JP3: footprint Jumper:SolderJumper-2_P1.3mm_Bridged_RoundedPad1.0x1.5mm -> Jumper:SolderJumper-2_P1.3mm_Open_RoundedPad1.0x1.5mm
- L1: value SRP3212A-2R2M -> 3.3uH; Height 1.2 -> 1; LCSC C22388372 -> C337905; Manufacturer_Name Bourns -> Murata Electronics; Manufacturer_Part_Number SRP3212A-3R3M -> 1277AS-H-3R3M=P2; Mouser Part Number 652-SRP3212A-3R3M -> 81-1277AS-H-3R3MP2; Mouser Price/Stock https://www.mouser.co.uk/ProductDetail/Bourns/SRP3212A-3R3M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 -> (none)
- L2: value SRP3212A-3R3M -> 4.7uH; Description_1 Ind,3.2x2.5x1mm,3.3uH+/-20%,3.1A,shd -> Ind,3.2x2.5x1mm,4.7uH+/-20%,3.1A,shd; Height 1.2 -> 1; LCSC C19779117 -> C1330201; Manufacturer_Name Bourns -> Murata; Manufacturer_Part_Number SRP3212A-3R3M -> 1276AS-H-4R7M=P2; Mouser Part Number 652-SRP3212A-3R3M -> 81-1276AS-H-4R7MP2; Mouser Price/Stock https://www.mouser.co.uk/ProductDetail/Bourns/SRP3212A-3R3M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 -> (none)
- R1, R11, R13, R14, R15, R18, R19, R2, R4, R5, R6, R7, R8, R9: footprint Resistor_SMD:R_1206_3216Metric -> Resistor_SMD:R_0805_2012Metric
- R3: footprint Resistor_SMD:R_1206_3216Metric -> Resistor_SMD:R_0805_2012Metric; LCSC C2849334 -> C422816
- Y1: LCSC C1985542 -> C1986264
Connections:
- net A0: now also IC5.5 (SDA); no longer IC5.1 (A0)
- net A1: now also IC5.6 (SCL); no longer IC5.2 (A1)
- net A2: now also IC5.7 (WP); no longer IC5.3 (A2)
- net GND: now also IC5.8 (VDD); no longer IC5.4 (VSS)
- net SCL1: now also IC5.2 (A1); no longer IC5.6 (SCL)
- net SDA1: now also IC5.1 (A0); no longer IC5.5 (SDA)
- net Write Protect: now also IC5.3 (A2); no longer IC5.7 (WP)
- net at C4.1, J16.2 (C), JP6.2 (B)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: now also IC5.4 (VSS); no longer IC5.8 (VDD)
Other:
- moved on the sheet: IC5
