File: LCC-Pico-Node_v3_0C - 0805.kicad_sch (KiCad schematic)
At the start: 85 parts, among them IC1 TPS54228DR, IC2 MCP2518FD, IC3 MCP2562FD, IC5 256Kb, IC6 TPS54228DR, J1 RJ45, J12 Power Sel, J15 Analog I/O, J16 NVM Power Sel, J2 RJ45, J20 Barrel Jack, J21 I/O - 1, J24 Ext. Reset, J27 MasterPower, J3 LCC Pwr Sel, J4 I/O - 2, J5 External Power, J6 Power Sel, J7 External Power, Q1 DMG2305UX-7, SW1 button, SW2 button, SW3 button, Y1 ABM-40MHZ

Commit message: fixed bad EEPROM footprint rotation
had rotated EEPROM incorrectly, this fixes it
Connections:
- net A0: now also IC5.1 (A0); no longer IC5.5 (SDA)
- net A1: now also IC5.2 (A1); no longer IC5.6 (SCL)
- net A2: now also IC5.3 (A2); no longer IC5.7 (WP)
- net GND: now also IC5.4 (VSS); no longer IC5.8 (VDD)
- net SCL1: now also IC5.6 (SCL); no longer IC5.2 (A1)
- net SDA1: now also IC5.5 (SDA); no longer IC5.1 (A0)
- net Write Protect: now also IC5.7 (WP); no longer IC5.3 (A2)
- net at C4.1, J16.2 (C), JP6.2 (B)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: now also IC5.8 (VDD); no longer IC5.4 (VSS)
Other:
- moved on the sheet: IC5
Changed lines of the file:
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@@
 	)
 	(junction
-		(at 66.04 190.5)
+		(at 22.86 43.18)
 		(diameter 0)
 		(color 0 0 0 0)
 	)
 	(junction
-		(at 69.85 74.93)
+		(at 66.04 190.5)
 		(diameter 0)
 		(color 0 0 0 0)
 	)
 	(junction
-		(at 36.83 163.83)
+		(at 69.85 74.93)
 		(diameter 0)
 		(color 0 0 0 0)
 	)
 	(junction
-		(at 69.85 93.98)
+		(at 36.83 163.83)
 		(diameter 0)
 		(color 0 0 0 0)
 	)
 	(junction
-		(at 22.86 43.18)
+		(at 69.85 93.98)
 		(diameter 0)
 		(color 0 0 0 0)
@@
 	(symbol
 		(lib_id "SamacSys_Parts:MB85RC256VPNF-G-JNE1")
-		(at 48.26 43.18 180)
+		(at 22.86 35.56 0)
 		(unit 1)
 		(exclude_from_sim no)
@@
 		(on_board yes)
 		(dnp no)
-		(fields_autoplaced yes)
 		(property "Reference" "IC5"
-			(at 35.56 27.94 0)
+			(at 35.56 50.8 0)
 			(effects
 				(font
@@
 		)
 		(property "Value" "256Kb"
-			(at 35.56 30.48 0)
+			(at 35.56 48.26 0)
 			(effects
 				(font
@@
 		)
 		(property "Footprint" "SamacSys_Parts:SOIC127P600X175-8N"
-			(at 26.67 45.72 0)
+			(at 44.45 33.02 0)
 			(effects
 				(font
@@
 		)
 		(property "Datasheet" "https://fscdn.rohm.com/en/products/databook/datasheet/ic/memory/eeprom/br24g256xxx-5-e.pdf"
-			(at 26.67 43.18 0)
+			(at 44.45 35.56 0)
 			(effects
 				(font
@@
 		)
 		(property "Description" "EEPROM ICs, Memory, 256KBit, I&sup2;C BUS, High Endurance, Low Power Serial EEPROM"
-			(at 48.26 43.18 0)
+			(at 22.86 35.56 0)
 			(effects
 				(font
@@
 		)
 		(property "Description_1" "EEPROM ICs, Memory, 256KBit, I&sup2;C BUS, High Endurance, Low Power Serial EEPROM "
-			(at 26.67 40.64 0)
+			(at 44.45 38.1 0)
 			(effects
 				(font
@@
 		)
 		(property "Height" "1.75"
-			(at 26.67 38.1 0)
+			(at 44.45 40.64 0)
 			(effects
 				(font
@@
 		)
 		(property "Mouser Part Number" "755-BR24G256F-5E2 "
-			(at 26.67 35.56 0)
+			(at 44.45 43.18 0)
 			(effects
 				(font
@@
 		)
 		(property "Mouser Price/Stock" "https://www.mouser.com/ProductDetail/ROHM-Semiconductor/BR24G256F-5E2?qs=PzGy0jfpSMt%2F62ePk7MQng%3D%3D"
-			(at 26.67 33.02 0)
+			(at 44.45 45.72 0)
 			(effects
 				(font
@@
 		)
 		(property "Manufacturer_Name" "ROHM Semiconductor "
-			(at 26.67 30.48 0)
+			(at 44.45 48.26 0)
 			(effects
 				(font
@@
 		)
 		(property "Manufacturer_Part_Number" "BR24G256F-5E2 "
-			(at 26.67 27.94 0)
+			(at 44.45 50.8 0)
 			(effects
 				(font
@@
 		)
 		(property "LCSC" "C90485"
-			(at 35.56 50.8 0)
+			(at 35.56 27.94 0)
 			(effects
 				(font
