File: LCC-Pico-Node_v3_0C - 1206.kicad_sch (KiCad schematic)
At the start: 85 parts, among them IC1 TPS54228DR, IC2 MCP2518FD, IC3 MCP2562FD, IC5 MB85RCxxxV, IC6 TPS54228DR, J1 RJ45, J12 Power Sel, J15 Analog I/O, J16 NVM Power Sel, J2 RJ45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

Commit message: Production level
0805 boards can be assembled at JLCPCB with these files
1206 boards are for hand assembly
Parts:
- L1: value SRP3212A-2R2M -> 3.3uH; Height 1.2 -> 1; LCSC C22388372 -> (none); Manufacturer_Name Bourns -> Murata Electronics; Manufacturer_Part_Number SRP3212A-3R3M -> 1277AS-H-3R3M=P2; Mouser Part Number 652-SRP3212A-3R3M -> 81-1277AS-H-3R3MP2; Mouser Price/Stock https://www.mouser.co.uk/ProductDetail/Bourns/SRP3212A-3R3M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 -> (none)
- L2: value SRP3212A-3R3M -> 4.7uH; Description_1 Ind,3.2x2.5x1mm,3.3uH+/-20%,3.1A,shd -> Ind,3.2x2.5x1mm,4.7uH+/-20%,3.1A,shd; Height 1.2 -> 1; LCSC C19779117 -> (none); Manufacturer_Name Bourns -> Murata; Manufacturer_Part_Number SRP3212A-3R3M -> 1276AS-H-4R7M=P2; Mouser Part Number 652-SRP3212A-3R3M -> 81-1276AS-H-4R7MP2; Mouser Price/Stock https://www.mouser.co.uk/ProductDetail/Bourns/SRP3212A-3R3M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 -> (none)
Changed lines of the file:
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@@
 			)
 		)
-		(property "Value" "SRP3212A-2R2M"
+		(property "Value" "3.3uH"
 			(at 83.82 184.658 0)
 			(effects
@@
 			)
 		)
-		(property "Datasheet" "https://www.bourns.com/docs/product-datasheets/srp3212.pdf"
+		(property "Datasheet" "https://www.mouser.com/datasheet/3/76/2/J_E_TE243A_0008.pdf"
 			(at 82.55 190.5 0)
 			(effects
@@
 			)
 		)
-		(property "Height" "1.2"
+		(property "Height" "1"
 			(at 87.63 190.5 0)
 			(effects
@@
 			)
 		)
-		(property "Mouser Part Number" "652-SRP3212A-3R3M"
+		(property "Mouser Part Number" "81-1277AS-H-3R3MP2"
 			(at 90.17 190.5 0)
 			(effects
@@
 			)
 		)
-		(property "Mouser Price/Stock" "https://www.mouser.co.uk/ProductDetail/Bourns/SRP3212A-3R3M?qs=t7xnP681wgXp9Q%252BFP%252BQamQ%3D%3D"
+		(property "Mouser Price/Stock" ""
 			(at 92.71 190.5 0)
 			(effects
@@
 			)
 		)
-		(property "Manufacturer_Name" "Bourns"
+		(property "Manufacturer_Name" "Murata Electronics"
 			(at 95.25 190.5 0)
 			(effects
@@
 			)
 		)
-		(property "Manufacturer_Part_Number" "SRP3212A-3R3M"
+		(property "Manufacturer_Part_Number" "1277AS-H-3R3M=P2"
 			(at 97.79 190.5 0)
 			(effects
@@
 			)
 		)
-		(property "LCSC" "C22388372"
+		(property "LCSC" ""
 			(at 80.518 184.15 0)
 			(effects
@@
 		)
 		(instances
-			(project "LCC-Pico-Node_v3_0 - 1206"
+			(project "LCC-Pico-Node_v3_0C - 1206"
 				(path "/e3a6af99-7545-47ae-86bc-5ee23a6e5e7d"
 					(reference "L1")
@@
 			)
 		)
-		(property "Value" "SRP3212A-3R3M"
+		(property "Value" "4.7uH"
 			(at 155.448 186.182 0)
 			(effects
@@
 			)
 		)
-		(property "Datasheet" "https://www.bourns.com/docs/product-datasheets/srp3212.pdf"
+		(property "Datasheet" "https://www.mouser.com/datasheet/3/76/2/J_E_TE243A_0009.pdf"
 			(at 152.4 191.77 0)
 			(effects
@@
 			)
 		)
-		(property "Description" "Ind,3.2x2.5x1mm,3.3uH+/-20%,3.1A,shd"
+		(property "Description" "Ind,3.2x2.5x1mm,4.7uH+/-20%,3.1A,shd"
 			(at 153.67 175.26 0)
 			(effects
@@
 			)
 		)
-		(property "Description_1" "Ind,3.2x2.5x1mm,3.3uH+/-20%,3.1A,shd"
+		(property "Description_1" "Ind,3.2x2.5x1mm,4.7uH+/-20%,3.1A,shd"
 			(at 149.86 191.77 0)
 			(effects
@@
 			)
 		)
-		(property "Height" "1.2"
+		(property "Height" "1"
 			(at 147.32 191.77 0)
 			(effects
@@
 			)
 		)
-		(property "Mouser Part Number" "652-SRP3212A-3R3M"
+		(property "Mouser Part Number" "81-1276AS-H-4R7MP2 "
 			(at 144.78 191.77 0)
 			(effects
@@
 			)
 		)
-		(property "Mouser Price/Stock" "https://www.mouser.co.uk/ProductDetail/Bourns/SRP3212A-3R3M?qs=t7xnP681wgXp9Q%252BFP%252BQamQ%3D%3D"
+		(property "Mouser Price/Stock" ""
 			(at 142.24 191.77 0)
 			(effects
@@
 			)
 		)
-		(property "Manufacturer_Name" "Bourns"
+		(property "Manufacturer_Name" "Murata"
 			(at 139.7 191.77 0)
 			(effects
@@
 			)
 		)
-		(property "Manufacturer_Part_Number" "SRP3212A-3R3M"
+		(property "Manufacturer_Part_Number" "1276AS-H-4R7M=P2 "
 			(at 137.16 191.77 0)
 			(effects
@@
 			)
 		)
-		(property "LCSC" "C19779117"
+		(property "LCSC" ""
 			(at 150.876 186.182 0)
 			(effects
@@
 		)
 		(instances
-			(project "LCC-Pico-Node_v3_0 - 1206"
+			(project "LCC-Pico-Node_v3_0C - 1206"
 				(path "/e3a6af99-7545-47ae-86bc-5ee23a6e5e7d"
 					(reference "L2")
