File: LCC-Pico-Node_v3_0C - 1206.kicad_sch (KiCad schematic)
At the start: 85 parts, among them IC1 TPS54228DR, IC2 MCP2518FD, IC3 MCP2562FD, IC5 MB85RCxxxV, IC6 TPS54228DR, J1 RJ45, J12 Power Sel, J15 Analog I/O, J16 NVM Power Sel, J2 RJ45, J20 Barrel Jack, J21 I/O - 1, J24 Ext. Reset, J27 MasterPower, J3 LCC Pwr Sel, J4 I/O - 2, J5 External Power, J6 Power Sel, J7 External Power, Q1 DMG2305UX-7, SW1 button, SW2 button, SW3 button, Y1 ABM-40MHZ

Commit message: barrel jack footprint fix
bad footprint replaced
Connections:
- net GND: no longer J20.3
- no-connect marks 8 -> 9
Changed lines of the file:
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@@
-	)
-	(junction
-		(at 36.83 163.83)
-		(diameter 0)
-		(color 0 0 0 0)
 	)
 	(junction
@@
 	)
 	(no_connect
+		(at 26.67 163.83)
+	)
+	(no_connect
 		(at 175.26 88.9)
 	)
@@
 		)
 		(stroke
-			(width 0)
-			(type default)
-		)
-	)
-	(wire
-		(pts
-			(xy 26.67 163.83) (xy 36.83 163.83)
-		)
-		(stroke
