File: RibbonBreakout2.kicad_pcb (KiCad board)
At the start: 2 copper layers, 31.5 x 38.6 mm, 13 parts

Commit message: Add Display090AdapterB & update gerbers
Replace Display090Adapter with a new Display090AdapterB set (new .kicad_pcb/.kicad_pro and updated .kicad_prl/.kicad_sch). Update RibbonBreakout and RibbonBreakout2 board files. Remove many individual gerber output files and add consolidated GERBER-*.zip archives under gerbers/. Also remove temporary/backup documentation files. These changes package gerbers and introduce the B revision of the 090 adapter.
Other:
- board text added: "GND +5v Data GND"
Changed lines of the file:
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@@
 		(layer "Edge.Cuts")
 	)
-	(gr_text "GND Data +5v GND"
+	(gr_text "GND +5v Data GND"
 		(at 142.4 113.9 0)
 		(layer "F.SilkS")
@@
 	)
 	(gr_text "GND Data +5v GND"
-		(at 142.2 78.8 0)
+		(at 154 78.35 180)
 		(layer "F.SilkS")
 		(effects
