File: RibbonBreakout_v2_7.kicad_pcb (KiCad board)
At the start: 2 copper layers, 30 x 40 mm, 22 parts, among them J1 Conn_01x10, J21 Node

Commit message: Add Display090AdapterB & update gerbers
Replace Display090Adapter with a new Display090AdapterB set (new .kicad_pcb/.kicad_pro and updated .kicad_prl/.kicad_sch). Update RibbonBreakout and RibbonBreakout2 board files. Remove many individual gerber output files and add consolidated GERBER-*.zip archives under gerbers/. Also remove temporary/backup documentation files. These changes package gerbers and introduce the B revision of the 090 adapter.
Routing:
- net GND: track 16.0 -> 54.9 mm, vias 9 -> 6
Other:
- board text added: "Rev B"
Changed lines of the file:
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@@
+		)
+	)
+	(gr_text "Rev B"
+		(at 143.75 118.4 0)
+		(layer "F.SilkS")
+		(effects
+			(font
+				(size 1 1)
+				(thickness 0.15)
+			)
+			(justify left bottom)
 		)
 	)
@@
 	)
 	(segment
+		(start 147.451 102.451)
+		(end 143.63 98.63)
+		(width 0.35)
+		(layer "F.Cu")
+		(net 2)
+	)
+	(segment
 		(start 155.03 96.01)
 		(end 151.9425 96.01)
@@
 	)
 	(segment
+		(start 151.9875 101.2)
+		(end 150.7365 102.451)
+		(width 0.35)
+		(layer "F.Cu")
+		(net 2)
+	)
+	(segment
+		(start 143.63 98.63)
+		(end 137.5 98.63)
+		(width 0.35)
+		(layer "F.Cu")
+		(net 2)
+	)
+	(segment
+		(start 150.7365 102.451)
+		(end 147.451 102.451)
+		(width 0.35)
+		(layer "F.Cu")
+		(net 2)
+	)
+	(segment
 		(start 158.4 99.38)
 		(end 155.03 96.01)
@@
 	)
 	(via
-		(at 151.8875 93.31)
-		(size 0.6)
-		(drill 0.3)
-		(layers "F.Cu" "B.Cu")
-		(net 2)
-	)
-	(via
 		(at 151.9875 109.22)
-		(size 0.6)
-		(drill 0.3)
-		(layers "F.Cu" "B.Cu")
-		(net 2)
-	)
-	(via
-		(at 151.9425 96.1)
-		(size 0.6)
-		(drill 0.3)
-		(layers "F.Cu" "B.Cu")
-		(net 2)
-	)
-	(via
-		(at 151.8875 111.9)
 		(size 0.6)
 		(drill 0.3)
@@
 	)
 	(segment
+		(start 158.4 99.38)
+		(end 156.37 97.35)
+		(width 0.35)
+		(layer "B.Cu")
+		(net 2)
+	)
+	(segment
 		(start 151.8875 87.9)
 		(end 151.8875 90.71)
@@
 	)
 	(segment
+		(start 156.37 97.35)
+		(end 138.65 97.35)
+		(width 0.35)
+		(layer "B.Cu")
+		(net 2)
+	)
+	(segment
 		(start 151.9875 106.5)
 		(end 151.9875 109.22)
 		(width 0.35)
 		(layer "B.Cu")
+		(net 2)
+	)
+	(segment
+		(start 138.65 97.48)
+		(end 137.5 98.63)
+		(width 0.35)
+		(layer "B.Cu")
+		(net 2)
+	)
+	(segment
+		(start 138.65 97.35)
+		(end 138.65 97.48)
+		(width 0.35)
+		(layer "B.Cu")
