File: LCC-Pico-Node_v3_0C - 0805.kicad_pcb (KiCad board)
At the start: 4 copper layers, 100 x 82 mm, 89 parts, among them IC1 TPS54228DR, IC2 MCP2518FD, IC3 MCP2562FD, IC5 256Kb, IC6 TPS54228DR, J1 RJ45, J12 Power Sel, J15 Analog I/O, J16 NVM Power Sel, J2 RJ45, J20 Barrel Jack, J21 I/O - 1, J24 Ext. Reset, J27 MasterPower, J3 LCC Pwr Sel, J4 I/O - 2, J5 External Power, J6 Power Sel, J7 External Power, Q1 DMG2305UX-7, SW1 button, SW2 button, SW3 button, Y1 ABM-40MHZ

Commit message: fixed bad EEPROM footprint rotation
had rotated EEPROM incorrectly, this fixes it
Parts:
- moved IC5 0.25 mm to (164.0, 77.5), turned to -90 degrees
Connections:
- C4 pad 1: Net-(IC5-VSS) -> Net-(IC5-VDD)
- IC5 pad 1: SDA1 -> A0
- IC5 pad 2: SCL1 -> A1
- IC5 pad 3: Write Protect -> A2
- IC5 pad 4: Net-(IC5-VSS) -> GND
- IC5 pad 5: A0 -> SDA1
- IC5 pad 6: A1 -> SCL1
- IC5 pad 7: A2 -> Write Protect
- IC5 pad 8: GND -> Net-(IC5-VDD)
- J16 pad 2: Net-(IC5-VSS) -> Net-(IC5-VDD)
- JP6 pad 2: Net-(IC5-VSS) -> Net-(IC5-VDD)
- JP7 pad 2: Net-(IC5-VSS) -> Net-(IC5-VDD)
- JP8 pad 2: Net-(IC5-VSS) -> Net-(IC5-VDD)
- JP9 pad 2: Net-(IC5-VSS) -> Net-(IC5-VDD)
- R13 pad 2: Net-(IC5-VSS) -> Net-(IC5-VDD)
- R14 pad 2: Net-(IC5-VSS) -> Net-(IC5-VDD)
Routing:
- net Net-(IC5-VSS): track 39.0 -> 0.00 mm, vias 2 -> 0
- net Net-(IC5-VDD): track 0.00 -> 39.0 mm, vias 0 -> 2
