File: LCC-Pico-Node_v3_0C - 1206.kicad_pcb (KiCad board)
At the start: 4 copper layers, 99.2 x 82 mm, 89 parts, among them IC1 TPS54228DR, IC2 MCP2518FD, IC3 MCP2562FD, IC5 MB85RCxxxV, IC6 TPS54228DR, J1 RJ45, J12 Power Sel, J15 Analog I/O, J16 NVM Power Sel, J2 RJ45, J20 Barrel Jack, J21 I/O - 1, J24 Ext. Reset, J27 MasterPower, J3 LCC Pwr Sel, J4 I/O - 2, J5 External Power, J6 Power Sel, J7 External Power, Q1 DMG2305UX-7, SW1 button, SW2 button, SW3 button, Y1 ABM-40MHZ

Commit message: barrel jack footprint fix
bad footprint replaced
Parts:
- L1: value SRP3212A-2R2M -> 3.3uH
- L2: value SRP3212A-3R3M -> 4.7uH
Routing:
- net VEXT: track 46.1 -> 47.1 mm
Changed lines of the file:
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@@
 	(net 85 "unconnected-(RPiPico1-3V3-Pad36)")
 	(net 86 "unconnected-(RPiPico1-3V3-Pad36)_1")
+	(net 87 "unconnected-(J20-Pad3)")
 	(footprint "SamacSys_Parts:SOT96P240X115-3N"
 		(layer "F.Cu")
@@
 			)
 		)
-		(property "Value" "SRP3212A-2R2M"
+		(property "Value" "3.3uH"
 			(at -0.49 -2.276 90)
 			(unlocked yes)
@@
 			)
 		)
-		(property "Datasheet" "https://www.bourns.com/docs/product-datasheets/srp3212.pdf"
+		(property "Datasheet" "https://www.mouser.com/datasheet/3/76/2/J_E_TE243A_0008.pdf"
 			(at 0 0 90)
 			(unlocked yes)
@@
 			)
 		)
-		(property "Height" "1.2"
+		(property "Height" "1"
 			(at 0 0 90)
 			(unlocked yes)
@@
 			)
 		)
-		(property "Mouser Part Number" "652-SRP3212A-3R3M"
+		(property "Mouser Part Number" "81-1277AS-H-3R3MP2"
 			(at 0 0 90)
 			(unlocked yes)
@@
 			)
 		)
-		(property "Mouser Price/Stock" "https://www.mouser.co.uk/ProductDetail/Bourns/SRP3212A-3R3M?qs=t7xnP681wgXp9Q%252BFP%252BQamQ%3D%3D"
+		(property "Mouser Price/Stock" ""
 			(at 0 0 90)
 			(unlocked yes)
@@
 			)
 		)
-		(property "Manufacturer_Name" "Bourns"
+		(property "Manufacturer_Name" "Murata Electronics"
 			(at 0 0 90)
 			(unlocked yes)
@@
 			)
 		)
-		(property "Manufacturer_Part_Number" "SRP3212A-3R3M"
+		(property "Manufacturer_Part_Number" "1277AS-H-3R3M=P2"
 			(at 0 0 90)
 			(unlocked yes)
@@
 			)
 		)
-		(property "LCSC" "C22388372"
+		(property "LCSC" ""
 			(at 0 0 90)
 			(unlocked yes)
@@
 		)
 		(pad "1" smd rect
-			(at -11.2 -5.6)
-			(size 2 2.2)
-			(layers "F.Cu" "F.Mask" "F.Paste")
-			(net 76 "VEXT")
-			(pintype "passive")
-		)
-		(pad "1" smd rect
 			(at -11.2 5.6)
 			(size 2 2.2)
@@
 			(pintype "passive")
 		)
+		(pad "3" smd rect
+			(at -11.2 -5.6)
+			(size 2 2.2)
+			(layers "F.Cu" "F.Mask" "F.Paste")
+			(net 87 "unconnected-(J20-Pad3)")
+			(pintype "passive+no_connect")
+		)
 		(embedded_fonts no)
 	)
@@
 			)
 		)
-		(property "Value" "SRP3212A-3R3M"
+		(property "Value" "4.7uH"
 			(at 3.2 -2.3625 90)
 			(unlocked yes)
@@
 			)
 		)
-		(property "Datasheet" "https://www.bourns.com/docs/product-datasheets/srp3212.pdf"
+		(property "Datasheet" "https://www.mouser.com/datasheet/3/76/2/J_E_TE243A_0009.pdf"
 			(at 0 0 90)
 			(unlocked yes)
@@
 			)
 		)
-		(property "Description" "Ind,3.2x2.5x1mm,3.3uH+/-20%,3.1A,shd"
+		(property "Description" "Ind,3.2x2.5x1mm,4.7uH+/-20%,3.1A,shd"
 			(at 0 0 90)
 			(unlocked yes)
@@
 			)
 		)
-		(property "Description_1" "Ind,3.2x2.5x1mm,3.3uH+/-20%,3.1A,shd"
+		(property "Description_1" "Ind,3.2x2.5x1mm,4.7uH+/-20%,3.1A,shd"
 			(at 0 0 90)
 			(unlocked yes)
@@
 			)
 		)
-		(property "Height" "1.2"
+		(property "Height" "1"
 			(at 0 0 90)
 			(unlocked yes)
@@
 			)
 		)
-		(property "Mouser Part Number" "652-SRP3212A-3R3M"
+		(property "Mouser Part Number" "81-1276AS-H-4R7MP2 "
 			(at 0 0 90)
 			(unlocked yes)
@@
 			)
 		)
-		(property "Mouser Price/Stock" "https://www.mouser.co.uk/ProductDetail/Bourns/SRP3212A-3R3M?qs=t7xnP681wgXp9Q%252BFP%252BQamQ%3D%3D"
+		(property "Mouser Price/Stock" ""
 			(at 0 0 90)
 			(unlocked yes)
@@
 			)
 		)
-		(property "Manufacturer_Name" "Bourns"
+		(property "Manufacturer_Name" "Murata"
 			(at 0 0 90)
 			(unlocked yes)
@@
 			)
 		)
-		(property "Manufacturer_Part_Number" "SRP3212A-3R3M"
+		(property "Manufacturer_Part_Number" "1276AS-H-4R7M=P2 "
 			(at 0 0 90)
 			(unlocked yes)
@@
 			)
 		)
-		(property "LCSC" "C19779117"
+		(property "LCSC" ""
 			(at 0 0 90)
 			(unlocked yes)
@@
 	)
 	(segment
-		(start 190.7 113.4)
-		(end 190.7 117.95)
-		(width 1)
-		(layer "F.Cu")
-		(net 76)
-	)
-	(segment
-		(start 188.1725 97.615)
-		(end 182.135 97.615)
-		(width 1)
-		(layer "F.Cu")
-		(net 76)
-	)
-	(segment
-		(start 188.9225 94.85)
+		(start 188.9225 93.8975)
 		(end 188.9225 88.995)
 		(width 1)
@@
 	)
 	(segment
-		(start 188.1725 97.615)
-		(end 188.1215 97.666)
+		(start 185.02 94.73)
+		(end 179.55 100.2)
 		(width 1)
 		(layer "F.Cu")
@@
 	)
 	(segment
-		(start 188.1725 108.815)
-		(end 194.3725 108.815)
+		(start 190.7 113.4)
+		(end 190.7 117.95)
 		(width 1)
 		(layer "F.Cu")
@@
 	)
 	(segment
-		(start 182.135 97.615)
-		(end 179.55 100.2)
+		(start 181.35 100.2)
+		(end 188.1725 107.0225)
 		(width 1)
 		(layer "F.Cu")
@@
 	)
 	(segment
-		(start 189.0425 94.73)
-		(end 188.9225 94.85)
-		(width 0.5)
+		(start 189.755 94.73)
+		(end 185.02 94.73)
+		(width 1)
 		(layer "F.Cu")
 		(net 76)
 	)
 	(segment
-		(start 188.1725 97.615)
-		(end 188.9225 96.865)
+		(start 189.755 94.73)
+		(end 188.9225 93.8975)
 		(width 1)
 		(layer "F.Cu")
@@
 	)
 	(segment
-		(start 188.9225 96.865)
-		(end 188.9225 94.85)
+		(start 179.55 100.2)
+		(end 181.35 100.2)
 		(width 1)
 		(layer "F.Cu")
@@
 	)
 	(segment
-		(start 188.1215 97.666)
-		(end 188.1215 108.764)
+		(start 188.1725 108.815)
+		(end 194.3725 108.815)
 		(width 1)
 		(layer "F.Cu")
@@
 	)
 	(segment
-		(start 188.1215 108.764)
+		(start 188.1725 107.0225)
 		(end 188.1725 108.815)
 		(width 1)
@@
 	)
 	(segment
-		(start 189.755 94.73)
-		(end 189.0425 94.73)
-		(width 0.5)
-		(layer "F.Cu")
-		(net 76)
-	)
-	(segment
 		(start 146.976 123.706)
 		(end 146.171 123.706)
@@
 		(net 84)
 	)
+	(segment
+		(start 188.1725 97.615)
+		(end 188.1215 97.666)
+		(width 1)
+		(layer "F.Cu")
+		(net 87)
+	)
 	(zone
